Commit message: Modified minor things and tested gmapping, move_base and Rviz

File: urdf/robot_laser_camera.xacro (robot description, xacro)
@@ -114,5 +114,5 @@
 		    <box size="0.025 0.025 0.025"/>
 	    </geometry>
-	    <material name="red">
+	    <material name="orange">
 		    <color rgba="1 0 0 1"/>
 	    </material>
@@ -136,5 +136,5 @@
 		    <box size="0.05 0.05 0.06"/>
 	    </geometry>
-	    <material name="red">
+	    <material name="blue">
 		    <color rgba="1 0 0 1"/>
 	    </material>
@@ -158,5 +158,5 @@
 		      <box size="0.025 0.025 0.025"/>
 	      </geometry>
-	      <material name="red">
+	      <material name="grey">
 		      <color rgba="1 0 0 1"/>
 	      </material>
@@ -186,5 +186,4 @@
   </joint>
   <joint name="hokuyo_joint" type="fixed">
-	  <axis xyz="0 1 0" />
 	  <origin xyz="0.12 0 0.0125" rpy="0 0 0"/>
 	  <parent link="link_chassis"/>
@@ -198,5 +197,4 @@
 	 </joint>
    <joint name="camera_joint" type="fixed">
-	  <axis xyz="0 1 0" />
 	  <origin xyz="0.02 0 0.055" rpy="0 0 0"/>
 	  <parent link="camera_support_link"/>

Commit message: Added more logfiles and fixed the problem with sending goals
The robot movement and the approachment to the ball must be fixed too

File: urdf/robot_laser_camera.xacro (robot description, xacro)
@@ -141,7 +141,7 @@
 	  </visual>
 	  <inertial>
-	    <mass value="1e-5" />
-	    <origin xyz="0 0 0" rpy="0 0 0"/>
-	    <inertia ixx="1e-6" ixy="0" ixz="0" iyy="1e-6" iyz="0" izz="1e-6" />
+	    <mass value="0.025"/>
+  		<origin xyz="0 0 0" rpy="0 0 0" />
+  		<inertia ixx="1.2708333e-5" ixy="0" ixz="0" iyy="1.0416667e-5" iyz="0" izz="1.2708333e-5"/>
 	  </inertial>
   </link>
@@ -170,5 +170,5 @@
   <!-- Joints -->
   <joint name="joint_right_wheel" type="continuous">
-    <origin rpy="0 0 0" xyz="-0.025 0.075 0"/>
+    <origin rpy="0 0 0" xyz="-0.075 0.075 0"/>
     <child link="link_right_wheel"/>
     <parent link="link_chassis"/>
@@ -178,5 +178,5 @@
   </joint>
   <joint name="joint_left_wheel" type="continuous">
-    <origin rpy="0 0 0" xyz="-0.025 -0.075 0"/>
+    <origin rpy="0 0 0" xyz="-0.075 -0.075 0"/>
     <child link="link_left_wheel"/>
     <parent link="link_chassis"/>
@@ -189,15 +189,14 @@
 	  <parent link="link_chassis"/>
 	  <child link="hokuyo_link"/>
-	 </joint>
+	</joint>
   <joint name="camera_support_joint" type="fixed">
-	  <axis xyz="0 1 0" />
-	  <origin xyz="0.06 0 0.0175" rpy="0 0 0"/>
+	  <origin xyz="0.08 0 0.0175" rpy="0 0 0"/>
 	  <parent link="link_chassis"/>
 	  <child link="camera_support_link"/>
-	 </joint>
-   <joint name="camera_joint" type="fixed">
+	</joint>
+  <joint name="camera_joint" type="fixed">
 	  <origin xyz="0.02 0 0.055" rpy="0 0 0"/>
 	  <parent link="camera_support_link"/>
 	  <child link="camera_link"/>
-	 </joint>
+	</joint>
 </robot>

Commit message: Added the PLAY state and fixed the robot motion
Also fixed some code

File: urdf/robot_laser_camera.xacro (robot description, xacro)
@@ -136,7 +136,5 @@
 		    <box size="0.05 0.05 0.06"/>
 	    </geometry>
-	    <material name="blue">
-		    <color rgba="1 0 0 1"/>
-	    </material>
+	    <material name="blue"/>
 	  </visual>
 	  <inertial>
@@ -158,7 +156,5 @@
 		      <box size="0.025 0.025 0.025"/>
 	      </geometry>
-	      <material name="grey">
-		      <color rgba="1 0 0 1"/>
-	      </material>
+	      <material name="green"/>
 	    </visual>
 	    <inertial>
@@ -170,5 +166,5 @@
   <!-- Joints -->
   <joint name="joint_right_wheel" type="continuous">
-    <origin rpy="0 0 0" xyz="-0.075 0.075 0"/>
+    <origin rpy="0 0 0" xyz="-0.025 0.075 0"/>
     <child link="link_right_wheel"/>
     <parent link="link_chassis"/>
@@ -178,5 +174,5 @@
   </joint>
   <joint name="joint_left_wheel" type="continuous">
-    <origin rpy="0 0 0" xyz="-0.075 -0.075 0"/>
+    <origin rpy="0 0 0" xyz="-0.025 -0.075 0"/>
     <child link="link_left_wheel"/>
     <parent link="link_chassis"/>
